File: AD2S1200/mainAD2S1200.sch (EAGLE design)
At the start: 36 parts, among them IC1 OPA1013D, IC2 OPA1013D, Q1(9235.11QRTZ) 8.192, X1 22-23-2041

Commit message: Ok
Parts:
- added C9: 100n, rcl:C-EUC0805
- added CVGND: (no value), rcl:C-EUC0805
- added R0_PWR, RSHNT: (no value), resistor:R-EU_R0805
- added R2: (no value), resistor:R-TRIMM64X
- added SV3, SV4: (no value), con-ml:ML14
- added X2, X3, X4, X5: 22-23-2021, con-molex:22-23-2021
- added X7: 22-23-2041, con-molex:22-23-2041
Connections:
- new net N$15: SV4.2, U$1G$4.DB0
- new net N$18: SV4.4, U$1G$4.DB1
- new net N$21: SV4.6, U$1G$4.DB2
- new net N$22: SV4.12, U$1G$4.DB5
- new net N$23: SV4.14, U$1G$4.DB6
- new net N$24: SV4.8, U$1G$4.DB3
- new net N$25: SV4.10, U$1G$4.DB4
- new net N$26: SV3.5, U$1G$4.DB11/SO
- new net N$27: SV3.7, U$1G$4.DB10/SCLK
- new net N$28: SV3.9, U$1G$4.DB9
- new net N$29: SV3.11, U$1G$4.DB8
- new net N$30: SV3.13, U$1G$4.DB7
- new net N$31: SV4.11, U$1G$3.LOT
- new net N$32: SV4.7, U$1G$3.DIR
- new net N$33: SV4.9, U$1G$3.DOS
- new net N$34: SV4.5, U$1G$3.NM
- new net N$35: SV4.3, U$1G$3.B
- new net N$36: SV4.1, U$1G$3.A
- new net N$37: SV4.13, U$1G$3.CPO
- new net N$38: SV3.6, U$1G$2.!RD
- new net N$39: SV3.8, U$1G$2.!CS
- new net N$40: SV3.10, U$1G$2.!SAMPLE
- new net N$41: SV3.12, U$1G$2.!RDVEL
- new net N$42: SV3.14, U$1G$2.!SOE
- new net N$43: SV3.4, U$1G$2.!RESET
- new net N$44: SV3.2, U$1G$2.FS1
- new net N$45: SV3.3, U$1G$2.FS2
- new net N$46: CA_CO1.2, R2.S
- new net N$47: RSHNT.1, X3-2.S, X4-2.S
- new net N$48: CA1.+, CA2.1, CA3.1, PAM1.PVDD, PAM1.PVDD1, R0_PWR.1
- new net N$49: R0_PWR.2, X7-1.S
- new net N$50: U$1G$5.REFOUT
- net !EXC: now also X5-1.S; no longer CA_CO2.2
- net +5V: now also C9.1, X2-1.S, X7-2.S, X7-3.S; no longer CA1.+, CA2.1, CA3.1, PAM1.PVDD, PAM1.PVDD1
- net EXC: now also R2.E, X5-2.S; no longer CA_CO1.2
- net GND: now also C9.2, SV3.1, X2-2.S
- net GNDA: now also CA_CO2.2, CVGND.2, R2.A
- net N$14: now also CVGND.1
- net N$8: now also RSHNT.2, X4-1.S
- net N$9: now also X3-1.S
- net VDD: now also X7-4.S
Other:
- moved on the sheet: CA_CO1, CA_CO2
